File: drivers.sch (KiCad schematic (older format))
At the start: 37 parts, among them J2 A_CS, J3 A_SW, J4 B_CS, J5 B_SW, J6 C_CS, J7 C_SW, U4 IS32FL3738, U5 IS32FL3738, U6 IS32FL3738

Commit message: Add: Improved layout
Parts:
- removed TP3: A_INTB, TestPoint:TestPoint_Pad_D1.0mm, symbol Connector:TestPoint
- removed TP4: B_INTB, TestPoint:TestPoint_Pad_D1.0mm, symbol Connector:TestPoint
- removed TP5: C_INTB, TestPoint:TestPoint_Pad_D1.0mm, symbol Connector:TestPoint
- added C25, C26, C27: 0.47uF, Capacitor_SMD:C_0603_1608Metric, symbol Device:C
- added C28, C29, C30: 0.1uF, Capacitor_SMD:CP_Elec_5x5.4, symbol Device:CP
- C10, C11, C12, C13, C14, C15, C16, C17, C18, C19, C20, C21, C22, C23, C24, C7, C8, C9: footprint Capacitor_SMD:C_0805_2012Metric -> Capacitor_SMD:C_0603_1608Metric
- TP13: value SHUT -> SD
- TP14: value SDA -> DA
- TP15: value SCL -> CL
Connections:
- net GND: now also C25.1, C26.1, C27.1, C28.2, C29.2, C30.2
- net PP5V: now also C28.1, C29.1, C30.1
- net PP3V3 renamed +3V3
- net +3V3: now also C25.2, C26.2, C27.2
- no-connect marks 0 -> 3
Other:
- moved on the sheet: C10, C11, C12, C13, C14, C15, C16, C17, C18, C19, C20, C21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

Commit message: Add: Watch crystal, switches
Parts:
- added TP3: A5V, TestPoint:TestPoint_Pad_D1.0mm, symbol Connector:TestPoint
- added TP4: B5V, TestPoint:TestPoint_Pad_D1.0mm, symbol Connector:TestPoint
- added TP5: C5V, TestPoint:TestPoint_Pad_D1.0mm, symbol Connector:TestPoint
- U4, U5, U6: Vendor (none) -> Digi-Key; Vendor Price 10p (none) -> 1.53; Vendor Price 1p (none) -> 1.71; Vendor SKU (none) -> 706-1664-1-ND
Connections:
- net PP5V: now also TP3.1, TP4.1, TP5.1
Changed lines of the file:
@@
 F 3 "http://www.issi.com/WW/pdf/IS32FL3738.pdf" H 4400 3000 50  0001 C CNN
 F 4 "Matrix A" H 4550 2973 50  0000 C CNN "Matrix"
+F 5 "Digi-Key" H 4400 3000 50  0001 C CNN "Vendor"
+F 6 "1.53" H 4400 3000 50  0001 C CNN "Vendor Price 10p"
+F 7 "1.71" H 4400 3000 50  0001 C CNN "Vendor Price 1p"
+F 8 "706-1664-1-ND" H 4400 3000 50  0001 C CNN "Vendor SKU"
 	1    4400 3000
 	1    0    0    -1
@@
 F 3 "http://www.issi.com/WW/pdf/IS32FL3738.pdf" H 6950 3000 50  0001 C CNN
 F 4 "Matrix B" H 7100 2973 50  0000 C CNN "Matrix"
+F 5 "Digi-Key" H 6950 3000 50  0001 C CNN "Vendor"
+F 6 "1.53" H 6950 3000 50  0001 C CNN "Vendor Price 10p"
+F 7 "1.71" H 6950 3000 50  0001 C CNN "Vendor Price 1p"
+F 8 "706-1664-1-ND" H 6950 3000 50  0001 C CNN "Vendor SKU"
 	1    6950 3000
 	1    0    0    -1
@@
 F 3 "http://www.issi.com/WW/pdf/IS32FL3738.pdf" H 9400 2950 50  0001 C CNN
 F 4 "Matrix C" H 9550 2923 50  0000 C CNN "Matrix"
+F 5 "Digi-Key" H 9400 2950 50  0001 C CNN "Vendor"
+F 6 "1.53" H 9400 2950 50  0001 C CNN "Vendor Price 10p"
+F 7 "1.71" H 9400 2950 50  0001 C CNN "Vendor Price 1p"
+F 8 "706-1664-1-ND" H 9400 2950 50  0001 C CNN "Vendor SKU"
 	1    9400 2950
 	1    0    0    -1
@@
 NoConn ~ 6650 4000
 NoConn ~ 4100 4000
+$Comp
+L Connector:TestPoint TP5
+U 1 1 5E62D1C6
+P 9800 6150
+F 0 "TP5" V 9995 6222 50  0000 C CNN
+F 1 "C5V" V 9904 6222 50  0000 C CNN
+F 2 "TestPoint:TestPoint_Pad_D1.0mm" H 10000 6150 50  0001 C CNN
+F 3 "~" H 10000 6150 50  0001 C CNN
+	1    9800 6150
+	1    0    0    -1
+$EndComp
+Wire Wire Line
+	9800 6250 9800 6150
+$Comp
+L Connector:TestPoint TP4
+U 1 1 5E63F79C
+P 7350 6150
+F 0 "TP4" V 7545 6222 50  0000 C CNN
+F 1 "B5V" V 7454 6222 50  0000 C CNN
+F 2 "TestPoint:TestPoint_Pad_D1.0mm" H 7550 6150 50  0001 C CNN
+F 3 "~" H 7550 6150 50  0001 C CNN
+	1    7350 6150
+	1    0    0    -1
+$EndComp
+Wire Wire Line
+	7350 6250 7350 6150
+$Comp
+L Connector:TestPoint TP3
+U 1 1 5E650E23
+P 4750 6150
+F 0 "TP3" V 4945 6222 50  0000 C CNN
+F 1 "A5V" V 4854 6222 50  0000 C CNN
+F 2 "TestPoint:TestPoint_Pad_D1.0mm" H 4950 6150 50  0001 C CNN
+F 3 "~" H 4950 6150 50  0001 C CNN
+	1    4750 6150
+	1    0    0    -1
+$EndComp
+Wire Wire Line
+	4750 6250 4750 6150
 $EndSCHEMATC
