File: support.sch (KiCad schematic (older format))
At the start: 26 parts, among them J1 USB_B_Micro, Q1 S8050, Q2 S8050, U1 LD39015M33R, U2 CP2102N-A01-GQFN24

Commit message: Add: Improved layout
Parts:
- added J?: Conn_02x02_Odd_Even, Connector_Molex:Molex_Micro-Fit_3.0_43045-0400_2x02_P3.00mm_Horizontal, symbol Connector_Generic:Conn_02x02_Odd_Even
- TP10: value FT_TX -> TX
- TP11: value FT_RX -> RX
- TP8: value MCU_EN -> EN
- TP9: value MCU_B -> IO0
Other:
- moved on the sheet: C1, C2, TP1, TP2, U1
Changed lines of the file:
@@
 L power:GND #PWR0101
 U 1 1 5EA92373
-P 3050 3250
-F 0 "#PWR0101" H 3050 3000 50  0001 C CNN
-F 1 "GND" H 3055 3077 50  0000 C CNN
-F 2 "" H 3050 3250 50  0001 C CNN
-F 3 "" H 3050 3250 50  0001 C CNN
-	1    3050 3250
+P 3200 4350
+F 0 "#PWR0101" H 3200 4100 50  0001 C CNN
+F 1 "GND" H 3205 4177 50  0000 C CNN
+F 2 "" H 3200 4350 50  0001 C CNN
+F 3 "" H 3200 4350 50  0001 C CNN
+	1    3200 4350
 	1    0    0    -1
 $EndComp
@@
 L Device:C C2
 U 1 1 5EA92374
-P 3750 2750
-F 0 "C2" H 3865 2796 50  0000 L CNN
-F 1 "10uF/25V" H 3865 2705 50  0000 L CNN
-F 2 "Capacitor_SMD:C_0805_2012Metric" H 3788 2600 50  0001 C CNN
-F 3 "~" H 3750 2750 50  0001 C CNN
-F 4 "Mouser" H 3750 2750 50  0001 C CNN "Vendor"
-F 5 "0.069" H 3750 2750 50  0001 C CNN "Vendor Price 10p"
-F 6 "0.172" H 3750 2750 50  0001 C CNN "Vendor Price 1p"
-F 7 "963-TMK212BBJ106MG-T" H 3750 2750 50  0001 C CNN "Vendor SKU"
-	1    3750 2750
+P 3900 3850
+F 0 "C2" H 4015 3896 50  0000 L CNN
+F 1 "10uF/25V" H 4015 3805 50  0000 L CNN
+F 2 "Capacitor_SMD:C_0805_2012Metric" H 3938 3700 50  0001 C CNN
+F 3 "~" H 3900 3850 50  0001 C CNN
+F 4 "Mouser" H 3900 3850 50  0001 C CNN "Vendor"
+F 5 "0.069" H 3900 3850 50  0001 C CNN "Vendor Price 10p"
+F 6 "0.172" H 3900 3850 50  0001 C CNN "Vendor Price 1p"
+F 7 "963-TMK212BBJ106MG-T" H 3900 3850 50  0001 C CNN "Vendor SKU"
+	1    3900 3850
 	1    0    0    -1
 $EndComp
@@
 L Device:C C1
 U 1 1 5EA92375
-P 2150 2750
-F 0 "C1" H 2265 2796 50  0000 L CNN
-F 1 "10uF/25V" H 2265 2705 50  0000 L CNN
-F 2 "Capacitor_SMD:C_0805_2012Metric" H 2188 2600 50  0001 C CNN
-F 3 "~" H 2150 2750 50  0001 C CNN
-F 4 "Mouser" H 2150 2750 50  0001 C CNN "Vendor"
-F 5 "0.069" H 2150 2750 50  0001 C CNN "Vendor Price 10p"
-F 6 "0.172" H 2150 2750 50  0001 C CNN "Vendor Price 1p"
-F 7 "963-TMK212BBJ106MG-T" H 2150 2750 50  0001 C CNN "Vendor SKU"
-	1    2150 2750
-	1    0    0    -1
-$EndComp
-Wire Wire Line
-	2150 2600 2600 2600
-Wire Wire Line
-	3350 2600 3750 2600
+P 2300 3850
+F 0 "C1" H 2415 3896 50  0000 L CNN
+F 1 "10uF/25V" H 2415 3805 50  0000 L CNN
+F 2 "Capacitor_SMD:C_0805_2012Metric" H 2338 3700 50  0001 C CNN
+F 3 "~" H 2300 3850 50  0001 C CNN
+F 4 "Mouser" H 2300 3850 50  0001 C CNN "Vendor"
+F 5 "0.069" H 2300 3850 50  0001 C CNN "Vendor Price 10p"
+F 6 "0.172" H 2300 3850 50  0001 C CNN "Vendor Price 1p"
+F 7 "963-TMK212BBJ106MG-T" H 2300 3850 50  0001 C CNN "Vendor SKU"
+	1    2300 3850
+	1    0    0    -1
+$EndComp
+Wire Wire Line
+	2300 3700 2750 3700
+Wire Wire Line
+	3500 3700 3900 3700
 $Comp
 L power:GND #PWR0102
 U 1 1 5EA92376
-P 2150 3100
-F 0 "#PWR0102" H 2150 2850 50  0001 C CNN
-F 1 "GND" H 2155 2927 50  0000 C CNN
-F 2 "" H 2150 3100 50  0001 C CNN
-F 3 "" H 2150 3100 50  0001 C CNN
-	1    2150 3100
-	1    0    0    -1
-$EndComp
-Wire Wire Line
-	2150 3100 2150 2900
-Wire Wire Line
-	3750 2600 3750 2300
-Connection ~ 3750 2600
+P 2300 4200
+F 0 "#PWR0102" H 2300 3950 50  0001 C CNN
+F 1 "GND" H 2305 4027 50  0000 C CNN
+F 2 "" H 2300 4200 50  0001 C CNN
+F 3 "" H 2300 4200 50  0001 C CNN
+	1    2300 4200
+	1    0    0    -1
+$EndComp
+Wire Wire Line
+	2300 4200 2300 4000
+Wire Wire Line
+	3900 3700 3900 3400
+Connection ~ 3900 3700
 $Comp
 L Regulator_Linear:LD39015M33R U1
 U 1 1 5EA92372
-P 3050 2700
-F 0 "U1" H 3050 3042 50  0000 C CNN
-F 1 "LD39015M33R" H 3050 2951 50  0000 C CNN
-F 2 "Package_TO_SOT_SMD:SOT-23-5" H 3050 3025 50  0001 C CIN
-F 3 "http://www.st.com/resource/en/datasheet/ld39015.pdf" H 3050 2700 50  0001 C CNN
-F 4 "511-LD39015M33R" H 3050 2700 50  0001 C CNN "Vendor SKU"
-F 5 "Mouser" H 3050 2700 50  0001 C CNN "Vendor"
-F 6 "0.61" H 3050 2700 50  0001 C CNN "Vendor Price 10p"
-F 7 "0.72" H 3050 2700 50  0001 C CNN "Vendor Price 1p"
-	1    3050 2700
-	1    0    0    -1
-$EndComp
-Wire Wire Line
-	3050 3000 3050 3250
-Wire Wire Line
-	2750 2700 2600 2700
-Wire Wire Line
-	2600 2700 2600 2600
-Connection ~ 2600 2600
-Wire Wire Line
-	2600 2600 2750 2600
-Wire Wire Line
-	3750 2900 3750 3150
+P 3200 3800
+F 0 "U1" H 3200 4142 50  0000 C CNN
+F 1 "LD39015M33R" H 3200 4051 50  0000 C CNN
+F 2 "Package_TO_SOT_SMD:SOT-23-5" H 3200 4125 50  0001 C CIN
+F 3 "http://www.st.com/resource/en/datasheet/ld39015.pdf" H 3200 3800 50  0001 C CNN
+F 4 "511-LD39015M33R" H 3200 3800 50  0001 C CNN "Vendor SKU"
+F 5 "Mouser" H 3200 3800 50  0001 C CNN "Vendor"
+F 6 "0.61" H 3200 3800 50  0001 C CNN "Vendor Price 10p"
+F 7 "0.72" H 3200 3800 50  0001 C CNN "Vendor Price 1p"
+	1    3200 3800
+	1    0    0    -1
+$EndComp
+Wire Wire Line
+	3200 4100 3200 4350
+Wire Wire Line
+	2900 3800 2750 3800
+Wire Wire Line
+	2750 3800 2750 3700
+Connection ~ 2750 3700
+Wire Wire Line
+	2750 3700 2900 3700
+Wire Wire Line
+	3900 4000 3900 4250
 $Comp
 L power:GND #PWR0103
 U 1 1 5EA92377
-P 3750 3150
-F 0 "#PWR0103" H 3750 2900 50  0001 C CNN
-F 1 "GND" H 3755 2977 50  0000 C CNN
-F 2 "" H 3750 3150 50  0001 C CNN
-F 3 "" H 3750 3150 50  0001 C CNN
-	1    3750 3150
-	1    0    0    -1
-$EndComp
-Text Notes 2850 1750 0    100  ~ 0
+P 3900 4250
+F 0 "#PWR0103" H 3900 4000 50  0001 C CNN
+F 1 "GND" H 3905 4077 50  0000 C CNN
+F 2 "" H 3900 4250 50  0001 C CNN
+F 3 "" H 3900 4250 50  0001 C CNN
+	1    3900 4250
+	1    0    0    -1
+$EndComp
+Text Notes 3000 2850 0    100  ~ 0
 LDO
 $Comp
 L Connector:TestPoint TP1
 U 1 1 5EA92378
-P 4200 2300
-F 0 "TP1" H 4258 2418 50  0000 L CNN
-F 1 "3V3" H 4258 2327 50  0000 L CNN
-F 2 "TestPoint:TestPoint_Pad_D1.0mm" H 4400 2300 50  0001 C CNN
-F 3 "~" H 4400 2300 50  0001 C CNN
-	1    4200 2300
-	1    0    0    -1
-$EndComp
-Wire Wire Line
-	4200 2300 3750 2300
-Connection ~ 3750 2300
-Wire Wire Line
-	3750 2300 3750 2100
+P 4350 3400
+F 0 "TP1" H 4408 3518 50  0000 L CNN
+F 1 "3V3" H 4408 3427 50  0000 L CNN
+F 2 "TestPoint:TestPoint_Pad_D1.0mm" H 4550 3400 50  0001 C CNN
+F 3 "~" H 4550 3400 50  0001 C CNN
+	1    4350 3400
+	1    0    0    -1
+$EndComp
+Wire Wire Line
+	4350 3400 3900 3400
+Connection ~ 3900 3400
+Wire Wire Line
+	3900 3400 3900 3200
 $Comp
 L Connector:TestPoint TP2
 U 1 1 5EA92379
-P 4650 2300
-F 0 "TP2" H 4708 2418 50  0000 L CNN
-F 1 "GND" H 4708 2327 50  0000 L CNN
-F 2 "TestPoint:TestPoint_Pad_D1.0mm" H 4850 2300 50  0001 C CNN
-F 3 "~" H 4850 2300 50  0001 C CNN
-	1    4650 2300
-	1    0    0    -1
-$EndComp
-Wire Wire Line
-	4650 2300 4650 2450
+P 4800 3400
+F 0 "TP2" H 4858 3518 50  0000 L CNN
+F 1 "GND" H 4858 3427 50  0000 L CNN
+F 2 "TestPoint:TestPoint_Pad_D1.0mm" H 5000 3400 50  0001 C CNN
+F 3 "~" H 5000 3400 50  0001 C CNN
+	1    4800 3400
+	1    0    0    -1
+$EndComp
+Wire Wire Line
+	4800 3400 4800 3550
 $Comp
 L power:GND #PWR0104
 U 1 1 5DF6C945
-P 4650 2450
-F 0 "#PWR0104" H 4650 2200 50  0001 C CNN
-F 1 "GND" H 4655 2277 50  0000 C CNN
-F 2 "" H 4650 2450 50  0001 C CNN
-F 3 "" H 4650 2450 50  0001 C CNN
-	1    4650 2450
-	1    0    0    -1
-$EndComp
-Text GLabel 1850 2600 0    49   Input ~ 0
+P 4800 3550
+F 0 "#PWR0104" H 4800 3300 50  0001 C CNN
+F 1 "GND" H 4805 3377 50  0000 C CNN
+F 2 "" H 4800 3550 50  0001 C CNN
+F 3 "" H 4800 3550 50  0001 C CNN
+	1    4800 3550
+	1    0    0    -1
+$EndComp
+Text GLabel 2000 3700 0    49   Input ~ 0
 PP5V
 Wire Wire Line
-	2150 2600 1850 2600
-Connection ~ 2150 2600
+	2300 3700 2000 3700
+Connection ~ 2300 3700
 $Comp
 L power:+3.3V #PWR0105
 U 1 1 5EA80DF5
-P 3750 2100
-F 0 "#PWR0105" H 3750 1950 50  0001 C CNN
-F 1 "+3.3V" H 3765 2273 50  0000 C CNN
-F 2 "" H 3750 2100 50  0001 C CNN
-F 3 "" H 3750 2100 50  0001 C CNN
-	1    3750 2100
+P 3900 3200
+F 0 "#PWR0105" H 3900 3050 50  0001 C CNN
+F 1 "+3.3V" H 3915 3373 50  0000 C CNN
+F 2 "" H 3900 3200 50  0001 C CNN
+F 3 "" H 3900 3200 50  0001 C CNN
+	1    3900 3200
 	1    0    0    -1
 $EndComp
@@
 AR Path="/5EA5FEAD/5ECA669B" Ref="TP8"  Part="1"
 F 0 "TP8" H 3892 5726 50  0000 R CNN
-F 1 "MCU_EN" H 3892 5817 50  0000 R CNN
+F 1 "EN" H 3892 5817 50  0000 R CNN
 F 2 "TestPoint:TestPoint_Pad_D1.0mm" H 4150 5700 50  0001 C CNN
 F 3 "~" H 4150 5700 50  0001 C CNN
@@
 AR Path="/5EA5FEAD/5ECAD588" Ref="TP9"  Part="1"
 F 0 "TP9" H 4008 6818 50  0000 L CNN
-F 1 "MCU_B" H 4008 6727 50  0000 L CNN
+F 1 "IO0" H 4008 6727 50  0000 L CNN
 F 2 "TestPoint:TestPoint_Pad_D1.0mm" H 4150 6700 50  0001 C CNN
 F 3 "~" H 4150 6700 50  0001 C CNN
@@
 AR Path="/5EA5FEAD/5F1FE5B6" Ref="TP10"  Part="1"
 F 0 "TP10" H 10142 5426 50  0000 R CNN
-F 1 "FT_TX" H 10142 5517 50  0000 R CNN
+F 1 "TX" H 10142 5517 50  0000 R CNN
 F 2 "TestPoint:TestPoint_Pad_D1.0mm" H 10400 5400 50  0001 C CNN
 F 3 "~" H 10400 5400 50  0001 C CNN
@@
 AR Path="/5EA5FEAD/5F2042A2" Ref="TP11"  Part="1"
 F 0 "TP11" H 10592 5426 50  0000 R CNN
-F 1 "FT_RX" H 10592 5517 50  0000 R CNN
+F 1 "RX" H 10592 5517 50  0000 R CNN
 F 2 "TestPoint:TestPoint_Pad_D1.0mm" H 10850 5400 50  0001 C CNN
 F 3 "~" H 10850 5400 50  0001 C CNN
@@
 Text HLabel 10650 5300 1    50   Output ~ 0
 FT_RX
+$Comp
+L Connector_Generic:Conn_02x02_Odd_Even J?
+U 1 1 5EDA1126
+P 2300 1450
+F 0 "J?" H 2350 1667 50  0000 C CNN
+F 1 "Conn_02x02_Odd_Even" H 2350 1576 50  0000 C CNN
+F 2 "Connector_Molex:Molex_Micro-Fit_3.0_43045-0400_2x02_P3.00mm_Horizontal" H 2300 1450 50  0001 C CNN
+F 3 "~" H 2300 1450 50  0001 C CNN
+	1    2300 1450
+	1    0    0    -1
+$EndComp
 $EndSCHEMATC

Commit message: Add: Watch crystal, switches
Parts:
- removed J?: Conn_02x02_Odd_Even, Connector_Molex:Molex_Micro-Fit_3.0_43045-0400_2x02_P3.00mm_Horizontal, symbol Connector_Generic:Conn_02x02_Odd_Even
- added D5, D6: MBRA340, Diode_SMD:D_SMA, symbol Diode:MBRA340
- added F2: 2A, Fuse:Bourns_MF-MSMF260-2_Polyfuse_2.6A, symbol Device:Polyfuse
- added J8: Barrel_Jack, Connector_BarrelJack:BarrelJack_Wuerth_6941xx301002, symbol Connector:Barrel_Jack
- F1: footprint Fuse:Fuse_0805_2012Metric -> Fuse:Bourns_MF-MSMF260-2_Polyfuse_2.6A; Vendor (none) -> RS-Online; Vendor Price 100p (none) -> 0.27; Vendor Price 10p (none) -> 0.28; Vendor Price 1p (none) -> 0.28; Vendor SKU (none) -> 647-8257
- J1: footprint Connector_USB:USB_Micro-B_GCT_USB3076-30-A -> Connector_USB:USB_Micro-B_Molex-105017-0001
- U1: value LD39015M33R -> MIC5219-3.3YM5-TR; symbol Regulator_Linear:LD39015M33R -> Regulator_Linear:MIC5219-3.3YM5; Vendor Mouser -> RS-Online; Vendor SKU 511-LD39015M33R -> MIC5219-3.3YM5-TR
Connections:
- wire segments 88 -> 93
Other:
- note added: "Barrel DC Input"
Changed lines of the file:
@@
 Connection ~ 3900 3700
 $Comp
-L Regulator_Linear:LD39015M33R U1
+L Regulator_Linear:MIC5219-3.3YM5 U1
 U 1 1 5EA92372
 P 3200 3800
 F 0 "U1" H 3200 4142 50  0000 C CNN
-F 1 "LD39015M33R" H 3200 4051 50  0000 C CNN
+F 1 "MIC5219-3.3YM5-TR" H 3200 4051 50  0000 C CNN
 F 2 "Package_TO_SOT_SMD:SOT-23-5" H 3200 4125 50  0001 C CIN
-F 3 "http://www.st.com/resource/en/datasheet/ld39015.pdf" H 3200 3800 50  0001 C CNN
-F 4 "511-LD39015M33R" H 3200 3800 50  0001 C CNN "Vendor SKU"
-F 5 "Mouser" H 3200 3800 50  0001 C CNN "Vendor"
+F 3 "https://docs.rs-online.com/1253/0900766b8138542f.pdf" H 3200 3800 50  0001 C CNN
+F 4 "MIC5219-3.3YM5-TR" H 3200 3800 50  0001 C CNN "Vendor SKU"
+F 5 "RS-Online" H 3200 3800 50  0001 C CNN "Vendor"
 F 6 "0.61" H 3200 3800 50  0001 C CNN "Vendor Price 10p"
 F 7 "0.72" H 3200 3800 50  0001 C CNN "Vendor Price 1p"
@@
 F 0 "F1" V 8475 1700 50  0000 C CNN
 F 1 "2A" V 8566 1700 50  0000 C CNN
-F 2 "Fuse:Fuse_0805_2012Metric" H 8750 1500 50  0001 L CNN
+F 2 "Fuse:Bourns_MF-MSMF260-2_Polyfuse_2.6A" H 8750 1500 50  0001 L CNN
 F 3 "~" H 8700 1700 50  0001 C CNN
-F 4 "" H 8700 1700 50  0001 C CNN "Vendor"
-F 5 "" H 8700 1700 50  0001 C CNN "Vendor SKU"
-F 6 "" H 8700 1700 50  0001 C CNN "Vendor Price 10p"
-F 7 "" H 8700 1700 50  0001 C CNN "Vendor Price 1p"
+F 4 "RS-Online" H 8700 1700 50  0001 C CNN "Vendor"
+F 5 "647-8257" H 8700 1700 50  0001 C CNN "Vendor SKU"
+F 6 "0.28" H 8700 1700 50  0001 C CNN "Vendor Price 10p"
+F 7 "0.28" H 8700 1700 50  0001 C CNN "Vendor Price 1p"
+F 8 "0.27" H 8700 1700 50  0001 C CNN "Vendor Price 100p"
 	1    8700 1700
 	0    1    1    0
@@
 F 0 "J1" H 7057 2367 50  0000 C CNN
 F 1 "USB_B_Micro" H 7057 2276 50  0000 C CNN
-F 2 "Connector_USB:USB_Micro-B_GCT_USB3076-30-A" H 7150 1850 50  0001 C CNN
+F 2 "Connector_USB:USB_Micro-B_Molex-105017-0001" H 7150 1850 50  0001 C CNN
 F 3 "~" H 7150 1850 50  0001 C CNN
 F 4 "Farnell" H 7000 1900 50  0001 C CNN "Vendor"
@@
 Text Notes 2450 5100 0    100  ~ 0
 Boot Control Trickery
-Text GLabel 9050 1700 2    49   Input ~ 0
+Text GLabel 9800 1700 2    49   Input ~ 0
 PP5V
 Wire Wire Line
 	8400 1700 8550 1700
 Connection ~ 8400 1700
-Wire Wire Line
-	8850 1700 9050 1700
 $Comp
 L Connector:TestPoint TP?
@@
 	1    0    0    -1
 $EndComp
-Text GLabel 6800 4800 0    50   Input ~ 0
-PP5V
 $Comp
 L Connector:TestPoint TP?
@@
 FT_RX
 $Comp
-L Connector_Generic:Conn_02x02_Odd_Even J?
-U 1 1 5EDA1126
-P 2300 1450
-F 0 "J?" H 2350 1667 50  0000 C CNN
-F 1 "Conn_02x02_Odd_Even" H 2350 1576 50  0000 C CNN
-F 2 "Connector_Molex:Molex_Micro-Fit_3.0_43045-0400_2x02_P3.00mm_Horizontal" H 2300 1450 50  0001 C CNN
-F 3 "~" H 2300 1450 50  0001 C CNN
-	1    2300 1450
-	1    0    0    -1
-$EndComp
+L Connector:Barrel_Jack J8
+U 1 1 5E4B6C8E
+P 2600 1800
+F 0 "J8" H 2657 2125 50  0000 C CNN
+F 1 "Barrel_Jack" H 2657 2034 50  0000 C CNN
+F 2 "Connector_BarrelJack:BarrelJack_Wuerth_6941xx301002" H 2650 1760 50  0001 C CNN
+F 3 "~" H 2650 1760 50  0001 C CNN
+F 4 "RS-Online" H 2600 1800 50  0001 C CNN "Vendor"
+F 5 "0.74" H 2600 1800 50  0001 C CNN "Vendor Price 1p"
+F 6 "122-4879" H 2600 1800 50  0001 C CNN "Vendor SKU"
+	1    2600 1800
+	1    0    0    -1
+$EndComp
+Wire Wire Line
+	2900 1900 3400 1900
+$Comp
+L power:GND #PWR0165
+U 1 1 5E4BA335
+P 3400 1900
+F 0 "#PWR0165" H 3400 1650 50  0001 C CNN
+F 1 "GND" H 3405 1727 50  0000 C CNN
+F 2 "" H 3400 1900 50  0001 C CNN
+F 3 "" H 3400 1900 50  0001 C CNN
+	1    3400 1900
+	1    0    0    -1
+$EndComp
+Text GLabel 4650 1700 2    49   Input ~ 0
+PP5V
+Wire Wire Line
+	4650 1700 4350 1700
+$Comp
+L Diode:MBRA340 D5
+U 1 1 5E4CDCA2
+P 4200 1700
+F 0 "D5" H 4200 1450 50  0000 C CNN
+F 1 "MBRA340" H 4200 1550 50  0000 C CNN
+F 2 "Diode_SMD:D_SMA" H 4200 1525 50  0001 C CNN
+F 3 "https://www.onsemi.com/pub/Collateral/MBRA340T3-D.PDF" H 4200 1700 50  0001 C CNN
+	1    4200 1700
+	-1   0    0    1
+$EndComp
+Text Notes 2700 1150 0    100  ~ 0
+Barrel DC Input
+$Comp
+L Diode:MBRA340 D6
+U 1 1 5E4DDDFC
+P 9400 1700
+F 0 "D6" H 9400 1450 50  0000 C CNN
+F 1 "MBRA340" H 9400 1550 50  0000 C CNN
+F 2 "Diode_SMD:D_SMA" H 9400 1525 50  0001 C CNN
+F 3 "https://www.onsemi.com/pub/Collateral/MBRA340T3-D.PDF" H 9400 1700 50  0001 C CNN
+	1    9400 1700
+	-1   0    0    1
+$EndComp
+Wire Wire Line
+	8850 1700 9250 1700
+Wire Wire Line
+	9550 1700 9800 1700
+Text Label 6800 4800 2    50   ~ 0
+USB_5V
+$Comp
+L Device:Polyfuse F2
+U 1 1 5E7434FA
+P 3650 1700
+F 0 "F2" V 3425 1700 50  0000 C CNN
+F 1 "2A" V 3516 1700 50  0000 C CNN
+F 2 "Fuse:Bourns_MF-MSMF260-2_Polyfuse_2.6A" H 3700 1500 50  0001 L CNN
+F 3 "~" H 3650 1700 50  0001 C CNN
+F 4 "RS-Online" H 3650 1700 50  0001 C CNN "Vendor"
+F 5 "647-8257" H 3650 1700 50  0001 C CNN "Vendor SKU"
+F 6 "0.28" H 3650 1700 50  0001 C CNN "Vendor Price 10p"
+F 7 "0.28" H 3650 1700 50  0001 C CNN "Vendor Price 1p"
+F 8 "0.27" H 3650 1700 50  0001 C CNN "Vendor Price 100p"
+	1    3650 1700
+	0    1    1    0
+$EndComp
+Wire Wire Line
+	2900 1700 3500 1700
+Wire Wire Line
+	3800 1700 4050 1700
 $EndSCHEMATC
